Commit message: add new g1 urdf

File: urdf/g1/g1_12dof.urdf (robot description, URDF)
Before this commit: robot g1_12dof, 31 links, 30 joints
Links:
- removed link imu_in_pelvis
- removed link imu_in_torso
- added link imu_link
- added link waist_support_link, mass 0.001; visual mesh filename=meshes/waist_support_link.STL
- added link waist_yaw_fixed_link, mass 0.244; visual mesh filename=meshes/waist_yaw_link.STL
- link left_ankle_pitch_link: geometry visual mesh filename=meshes/left_ankle_pitch_link.STL
- link left_ankle_roll_link: geometry collision sphere radius=0.02; collision sphere radius=0.02
- link left_elbow_link: geometry visual mesh filename=meshes/left_elbow_link.STL
- link left_hip_pitch_link: geometry visual mesh filename=meshes/left_hip_pitch_link.STL
- link left_hip_roll_link: geometry visual mesh filename=meshes/left_hip_roll_link.STL
- link left_hip_yaw_link: geometry visual mesh filename=meshes/left_hip_yaw_link.STL
- link left_knee_link: geometry visual mesh filename=meshes/left_knee_link.STL
- link left_shoulder_pitch_link: geometry visual mesh filename=meshes/left_shoulder_pitch_link.STL
- link left_shoulder_roll_link: geometry visual mesh filename=meshes/left_shoulder_roll_link.STL
- link left_shoulder_yaw_link: geometry visual mesh filename=meshes/left_shoulder_yaw_link.STL
- link left_wrist_roll_rubber_hand: geometry visual mesh filename=meshes/left_wrist_roll_rubber_hand.STL
- link right_ankle_pitch_link: geometry visual mesh filename=meshes/right_ankle_pitch_link.STL
- link right_ankle_roll_link: geometry collision sphere radius=0.02; collision sphere radius=0.02
- link right_elbow_link: geometry visual mesh filename=meshes/right_elbow_link.STL
- link right_hip_pitch_link: geometry visual mesh filename=meshes/right_hip_pitch_link.STL
- link right_hip_roll_link: geometry visual mesh filename=meshes/right_hip_roll_link.STL
- link right_hip_yaw_link: geometry visual mesh filename=meshes/right_hip_yaw_link.STL
- link right_knee_link: geometry visual mesh filename=meshes/right_knee_link.STL
- link right_shoulder_pitch_link: geometry visual mesh filename=meshes/right_shoulder_pitch_link.STL
- link right_shoulder_roll_link: geometry visual mesh filename=meshes/right_shoulder_roll_link.STL
- link right_shoulder_yaw_link: geometry visual mesh filename=meshes/right_shoulder_yaw_link.STL
- link right_wrist_roll_rubber_hand: geometry visual mesh filename=meshes/right_wrist_roll_rubber_hand.STL
- link torso_link: mass 6.78 -> 8.562; geometry collision mesh filename=meshes/torso_link.STL; visual mesh filename=meshes/torso_link.STL
Joints:
- removed joint imu_in_pelvis_joint
- removed joint imu_in_torso_joint
- added joint imu_joint: type fixed, parent torso_link, child imu_link, origin xyz=-0.03959 -0.00224 0.13792 rpy=0 0 0
- added joint waist_support_joint: type fixed, parent torso_link, child waist_support_link, origin xyz=0.0039635 0 -0.054 rpy=0 0 0
- added joint waist_yaw_fixed_joint: type fixed, parent torso_link, child waist_yaw_fixed_link, origin xyz=0.0039635 0 -0.054 rpy=0 0 0
- joint d435_joint: origin xyz=0.0576235 0.01753 0.42987 rpy=0 0.8307767239493009 0 -> xyz=0.0576235 0.01753 0.41987 rpy=0 0.8307767239493009 0
- joint head_joint: origin xyz=0.0039635 0 -0.044 rpy=0 0 0 -> xyz=0.0039635 0 -0.054 rpy=0 0 0
- joint left_hip_roll_joint: limit lower=-0.5236 upper=2.9671 effort=139 velocity=20 -> lower=-0.5236 upper=2.9671 effort=88 velocity=32
- joint left_shoulder_pitch_joint: origin xyz=0.0039563 0.10022 0.24778 rpy=0.27931 5.4949E-05 -0.00019159 -> xyz=0.0039563 0.10022 0.23778 rpy=0.27931 5.4949E-05 -0.00019159
- joint logo_joint: origin xyz=0.0039635 0 -0.044 rpy=0 0 0 -> xyz=0.0039635 0 -0.054 rpy=0 0 0
- joint mid360_joint: origin xyz=0.0002835 0.00003 0.41618 rpy=0 0.04014257279586953 0 -> xyz=0.0002835 0.00003 0.40618 rpy=0 0.04014257279586953 0
- joint right_hip_roll_joint: limit lower=-2.9671 upper=0.5236 effort=139 velocity=20 -> lower=-2.9671 upper=0.5236 effort=88 velocity=32
- joint right_shoulder_pitch_joint: origin xyz=0.0039563 -0.10021 0.24778 rpy=-0.27931 5.4949E-05 0.00019159 -> xyz=0.0039563 -0.10021 0.23778 rpy=-0.27931 5.4949E-05 0.00019159
- joint waist_yaw_joint: origin xyz=-0.0039635 0 0.044 rpy=0 0 0 -> xyz=-0.0039635 0 0.054 rpy=0 0 0
