Commit message: URDF: simplified part of g1; Cfg: Good Reward.

File: Genesis/genesis/assets/urdf/g1/g1_12dof_full.urdf (robot description, URDF)
Before this commit: robot g1_12dof, 32 links, 31 joints
Links:
- link left_ankle_pitch_link: geometry visual mesh filename=meshes/left_ankle_pitch_link.STL
- link left_elbow_link: geometry visual mesh filename=meshes/left_elbow_link.STL
- link left_hip_pitch_link: geometry visual mesh filename=meshes/left_hip_pitch_link.STL
- link left_hip_roll_link: geometry visual mesh filename=meshes/left_hip_roll_link.STL
- link left_shoulder_pitch_link: geometry visual mesh filename=meshes/left_shoulder_pitch_link.STL
- link left_shoulder_roll_link: geometry visual mesh filename=meshes/left_shoulder_roll_link.STL
- link left_shoulder_yaw_link: geometry visual mesh filename=meshes/left_shoulder_yaw_link.STL
- link left_wrist_roll_rubber_hand: geometry visual mesh filename=meshes/left_wrist_roll_rubber_hand.STL
- link right_ankle_pitch_link: geometry visual mesh filename=meshes/right_ankle_pitch_link.STL
- link right_elbow_link: geometry visual mesh filename=meshes/right_elbow_link.STL
- link right_hip_pitch_link: geometry visual mesh filename=meshes/right_hip_pitch_link.STL
- link right_hip_roll_link: geometry visual mesh filename=meshes/right_hip_roll_link.STL
- link right_shoulder_pitch_link: geometry visual mesh filename=meshes/right_shoulder_pitch_link.STL
- link right_shoulder_roll_link: geometry visual mesh filename=meshes/right_shoulder_roll_link.STL
- link right_shoulder_yaw_link: geometry visual mesh filename=meshes/right_shoulder_yaw_link.STL
- link right_wrist_roll_rubber_hand: geometry visual mesh filename=meshes/right_wrist_roll_rubber_hand.STL

Commit message: update deploy; update g1_12dof_full

File: Genesis/genesis/assets/urdf/g1/g1_12dof_full.urdf (robot description, URDF)
Before this commit: robot g1_12dof, 32 links, 31 joints
Links:
- link left_knee_link: geometry collision cylinder length=0.2 radius=0.05; visual mesh filename=meshes/left_knee_link.STL
- link right_knee_link: geometry collision cylinder length=0.2 radius=0.05; visual mesh filename=meshes/right_knee_link.STL
