Commit message: clean agent_pose prompts

File: Genesis/genesis/assets/urdf/leap_hand/leap_hand_left_glb.urdf (robot description, URDF)
Before this commit: robot leap_left, 22 links, 21 joints
Links:
- removed link index_tip_head
- removed link middle_tip_head
- removed link ring_tip_head
- removed link thumb_tip_head
Joints:
- removed joint index_tip
- removed joint middle_tip
- removed joint ring_tip
- removed joint thumb_tip

File: Genesis/genesis/assets/urdf/leap_hand/leap_hand_right_glb.urdf (robot description, URDF)
Before this commit: robot leap_right, 22 links, 21 joints
Links:
- removed link index_tip_head
- removed link middle_tip_head
- removed link ring_tip_head
- removed link thumb_tip_head
Joints:
- removed joint index_tip
- removed joint middle_tip
- removed joint ring_tip
- removed joint thumb_tip
